File: Mangler.kicad_pcb (KiCad board)
At the start: 2 copper layers, 62 x 73.2 mm, 22 parts, among them J1 USB, J2 ICE 10pin, J3 ANALOG, J4 PWR/RESET, J5 DIGITAL, J6 I2C, J7 SPI, U1 TLV1963-33DGYR, U2 SAMD21G18A-AF, Y1 Crystal

Commit message: Pin updates
Pin location updates and pin labals on silkscreen
Connections:
- J5 pad 3: D2 -> GND
- J5 pad 4: D3 -> GND
- J5 pad 5: D4 -> GND
- J5 pad 8: D7 -> GND
- J5 pad 9: D8 -> GND
- J7 pad 2: MOSI -> SCK
- J7 pad 3: SCK -> MOSI
- U2 pad 11: D8 -> (no net)
- U2 pad 13: D4 -> (no net)
- U2 pad 14: D3 -> (no net)
- U2 pad 23: D2 -> (no net)
- U2 pad 30: D7 -> (no net)
Routing:
- net D3: track 120.0 -> 0.00 mm
- net D1: track 107.1 -> 43.4 mm, vias 0 -> 1
- net D4: track 57.0 -> 0.00 mm
- net D8: track 48.6 -> 0.00 mm
- net D2: track 45.4 -> 0.00 mm
- net D0: track 85.4 -> 41.2 mm, vias 0 -> 1
- net D7: track 19.5 -> 0.00 mm
- net D5: track 58.5 -> 43.4 mm
- net D9: track 48.6 -> 43.2 mm
- net MISO: track 32.3 -> 29.0 mm
- net MOSI: track 34.0 -> 37.1 mm
- net SCK: track 33.2 -> 31.9 mm
Other:
- board size 62 x 73.2 mm -> 62.5 x 73.2 mm
- board text added: "0 1 GND GND GND 5 6 GND GND 9 10 11 12 13"
- board text added: "A0/14 A1/15 A2/16 A3/17 A4/18 A5/19"
- board text added: "Vcc MISO MOSI SCK GND"
- board text added: "Vcc SCL SDA GND"
- board text added: "Vcc Vcc RESET GND GND"
