File: Mangler.sch (KiCad schematic (older format))
At the start: 22 parts, among them J1 USB, J2 ICE 10pin, J3 ANALOG, J4 PWR/RESET, J5 DIGITAL, J6 I2C, J7 SPI, U1 TLV1963-33DGYR, U2 SAMD21G18A-AF, Y1 Crystal

Commit message: Pin updates
Pin location updates and pin labals on silkscreen
Connections:
- net labels removed: D2, D3, D4, D7, D8
- wire segments 31 -> 37
- no-connect marks 11 -> 16
Changed lines of the file:
@@
 Text GLabel 2275 5600 0    50   Input ~ 0
 A4
-Text GLabel 2275 5700 0    50   Input ~ 0
-D8
 Text GLabel 2275 5800 0    50   Input ~ 0
 D9
@@
 NoConn ~ 3725 4250
 NoConn ~ 3825 4250
-Text GLabel 4375 5300 2    50   Input ~ 0
-D7
 Text GLabel 4375 5400 2    50   Input ~ 0
 D6
@@
 Text GLabel 3825 6300 3    50   Input ~ 0
 D5
-Text GLabel 3725 6300 3    50   Input ~ 0
-D2
 Text GLabel 3025 6300 3    50   Input ~ 0
 D0
@@
 Text GLabel 2925 6300 3    50   Input ~ 0
 D1
-Text GLabel 2825 6300 3    50   Input ~ 0
-D3
-Text GLabel 2725 6300 3    50   Input ~ 0
-D4
 NoConn ~ 3625 6300
 Text GLabel 3900 2225 1    50   Input ~ 0
@@
 Text GLabel 8800 4325 0    50   Input ~ 0
 D1
-Text GLabel 8800 4425 0    50   Input ~ 0
-D2
-Text GLabel 8800 4525 0    50   Input ~ 0
-D3
-Text GLabel 8800 4625 0    50   Input ~ 0
-D4
 Text GLabel 8800 4725 0    50   Input ~ 0
 D5
 Text GLabel 8800 4825 0    50   Input ~ 0
 D6
-Text GLabel 8800 4925 0    50   Input ~ 0
-D7
-Text GLabel 8800 5025 0    50   Input ~ 0
-D8
 Text GLabel 8800 5125 0    50   Input ~ 0
 D9
@@
 	1    0    0    -1
 $EndComp
+Text GLabel 7625 6075 0    50   Input ~ 0
+MOSI
 Text GLabel 7625 5975 0    50   Input ~ 0
-MOSI
-Text GLabel 7625 6075 0    50   Input ~ 0
 SCK
 Text GLabel 7625 6175 0    50   Input ~ 0
 MISO
+$Comp
+L power:GND #PWR0101
+U 1 1 5C40DC7F
+P 8500 4525
+F 0 "#PWR0101" H 8500 4275 50  0001 C CNN
+F 1 "GND" H 8505 4352 50  0000 C CNN
+F 2 "" H 8500 4525 50  0001 C CNN
+F 3 "" H 8500 4525 50  0001 C CNN
+	1    8500 4525
+	1    0    0    -1
+$EndComp
+Wire Wire Line
+	8800 4625 8800 4525
+Connection ~ 8800 4525
+Wire Wire Line
+	8800 4525 8800 4425
+Wire Wire Line
+	8800 4525 8500 4525
+Wire Wire Line
+	8800 5025 8800 4975
+$Comp
+L power:GND #PWR0102
+U 1 1 5C40ED13
+P 8500 4975
+F 0 "#PWR0102" H 8500 4725 50  0001 C CNN
+F 1 "GND" H 8505 4802 50  0000 C CNN
+F 2 "" H 8500 4975 50  0001 C CNN
+F 3 "" H 8500 4975 50  0001 C CNN
+	1    8500 4975
+	1    0    0    -1
+$EndComp
+Wire Wire Line
+	8500 4975 8800 4975
+Connection ~ 8800 4975
+Wire Wire Line
+	8800 4975 8800 4925
+NoConn ~ 4375 5300
+NoConn ~ 2275 5700
+NoConn ~ 2725 6300
+NoConn ~ 2825 6300
+NoConn ~ 3725 6300
 $EndSCHEMATC
